File: Rev_1/ECAD/main_board/equalizer_channel_a.kicad_sch (KiCad schematic)
At the start: 27 parts, among them U20 NE5532, U21 NE5532

Commit message: Probably finished with PCB
Parts:
- removed U20, U21: NE5532, Package_SO:SOIC-8_3.9x4.9mm_P1.27mm, symbol Amplifier_Operational:NE5532
- added TP11: FILTER 1, TestPoint:TestPoint_Pad_1.0x1.0mm, symbol Connector:TestPoint
- added TP12: FILTER 2, TestPoint:TestPoint_Pad_1.0x1.0mm, symbol Connector:TestPoint
- added U5, U6: OPA1652, Package_SO:JEITA_SOIC-8_3.9x4.9mm_P1.27mm, symbol filip:OPA1652
- C20: renamed from C29; ID (none) -> 41
- C21: renamed from C27; ID (none) -> 25
- C22: renamed from C30; ID (none) -> 25
- C23: renamed from C28; ID (none) -> 25
- C24: ID (none) -> 8
- C25: renamed from C31; ID (none) -> 25
- C26: renamed from C25; ID (none) -> 8
- C27: renamed from C26; ID (none) -> 8
- C28: renamed from C21; value 330n -> 27n
- C29: renamed from C22; ID (none) -> 39
- C30: renamed from C23; ID (none) -> 40
- R20: ID (none) -> 44
- R21, R23: ID (none) -> 14
- R22, R24: ID (none) -> 67
- R25: renamed from R29; ID (none) -> 43
- R26: renamed from R25; ID (none) -> 66
- R27: renamed from R30; ID (none) -> 46
- R28: renamed from R31; ID (none) -> 67
- R29: renamed from R26; ID (none) -> 14
- R30: renamed from R27; ID (none) -> 47
- R31: renamed from R32; ID (none) -> 47
- R32: renamed from R28; ID (none) -> 45
- renumbered C20 to C19
Connections:
- net -5V is gone; now on net GND: C22.1, C25.2
- net GND: now also U5.4 (V-), U6.4 (V-); no longer C20.1, C21.2, C22.2, C23.1, C25.1, C30.1, R20.2, R22.2, R25.1
- net INPUT_IMPEDANCE: now also U5.3 (+)
- net OUT: now also TP12.1, U6.6 (-), U6.7
- net at C26.2, R27.2, R31.2: now also U5.7
- net at C29.1, R30.2, R31.1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: now also TP11.1
- net at C30.2, R32.2: now also U6.5 (+)
- net at R21.1, R23.1: now also U5.2 (-)
- net at C24.1, R23.2, R24.1: now also U5.1
- net at C28.1, R26.2, R29.1: now also U6.2 (-)
- net at C28.2, R29.2, R30.1: now also U6.1
- net at C27.2, R28.1: now also U5.6 (-)
- net +5V renamed +8V
- net +8V: now also U5.8 (V+), U6.8 (V+)
- new net +4V: C20.1, C21.2, C22.2, C23.1, C25.1, C30.1, R20.2, R22.2, R25.1, U5.5 (+), U6.3 (+)

Commit message: Exported Gerber and IBOM
Parts:
- TP11, TP12: now left out of the parts list
Changed lines of the file:
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@@
 		(body_style 1)
 		(exclude_from_sim no)
-		(in_bom yes)
+		(in_bom no)
 		(on_board yes)
 		(in_pos_files yes)
@@
 		(body_style 1)
 		(exclude_from_sim no)
-		(in_bom yes)
-		(on_board yes)
-		(in_pos_files yes)
+		(in_bom no)
+		(on_board yes)
+		(in_pos_files yes)

Commit message: Finished with adding 9V Power Delivery
Parts:
- C19: ID (none) -> 94
- C28: ID (none) -> 95
- U5, U6: ID (none) -> 100
Changed lines of the file:
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@@
 			)
 		)
-		(property "ID" ""
+		(property "ID" "95"
 			(at 140.97 71.12 90)
 			(hide yes)
@@
 			)
 		)
-		(property "ID" ""
+		(property "ID" "94"
 			(at 43.18 90.17 90)
 			(hide yes)
@@
 			)
 		)
+		(property "ID" "100"
+			(at 63.5 59.69 0)
+			(hide yes)
+			(show_name no)
+			(do_not_autoplace no)
+			(effects
+				(font
+					(size 1.27 1.27)
+				)
+			)
+		)
 		(pin "2"
 		)
@@
 			)
 		)
+		(property "ID" "100"
+			(at 198.12 92.71 0)
+			(hide yes)
+			(show_name no)
+			(do_not_autoplace no)
+			(effects
+				(font
+					(size 1.27 1.27)
+				)
+			)
+		)
 		(pin "2"
 		)
@@
 			)
 		)
+		(property "ID" "100"
+			(at 143.51 135.89 0)
+			(hide yes)
+			(show_name no)
+			(do_not_autoplace no)
+			(effects
+				(font
+					(size 1.27 1.27)
+				)
+			)
+		)
 		(pin "7"
 		)
@@
 			)
 		)
+		(property "ID" "100"
+			(at 82.55 92.71 0)
+			(hide yes)
+			(show_name no)
+			(do_not_autoplace no)
+			(effects
+				(font
+					(size 1.27 1.27)
+				)
+			)
+		)
 		(pin "6"
 		)
@@
 			)
 		)
+		(property "ID" "100"
+			(at 100.33 59.69 0)
+			(hide yes)
+			(show_name no)
+			(do_not_autoplace no)
+			(effects
+				(font
+					(size 1.27 1.27)
+				)
+			)
+		)
 		(pin "8"
 		)
@@
 			(at 140.97 95.25 0)
 			(hide yes)
+			(show_name no)
+			(do_not_autoplace no)
+			(effects
+				(font
+					(size 1.27 1.27)
+				)
+			)
+		)
+		(property "ID" "100"
+			(at 140.97 95.25 0)
+			(hide yes)
