File: Rev_1/ECAD/main_board/equalizer_channel_b.kicad_sch (KiCad schematic)
At the start: 24 parts, among them U40 NE5532, U41 NE5532

Commit message: Semi finsihed schematic
Parts:
- added C49: 100p, Capacitor_SMD:C_0805_2012Metric, symbol Device:C_Small
- C40, C41, C42, C43, C44, C45, C46, C47, C48: footprint (none) -> Capacitor_SMD:C_0805_2012Metric
- R40+1: renamed from R40+; footprint (none) -> Resistor_SMD:R_0805_2012Metric
- R41, R42, R43, R44, R45, R46, R47, R48, R49, R50, R51, R52: footprint (none) -> Resistor_SMD:R_0805_2012Metric
- U40, U41: footprint (none) -> Package_SO:SOIC-8_5.3x6.2mm_P1.27mm
Connections:
- net GND: now also C49.1
- net at C40.2, R40+1.1, U40.3 (+): now also C49.2
Other:
- moved on the sheet: C40, C41, C42, C43, C44, C45, C46, C47, C48, R40+1, R41, R42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

Commit message: Finished
Parts:
- added C50, C51: 100n, Capacitor_SMD:C_0805_2012Metric, symbol Device:C
- U40, U41: footprint Package_SO:SOIC-8_5.3x6.2mm_P1.27mm -> Package_SO:SOIC-8_3.9x4.9mm_P1.27mm; Mouser No: (none) -> 595-NE5532DR
- renumbered R40+1 to R40
Connections:
- net +5V: now also C50.2; no longer C48.1
- net -5V: now also C48.1, C51.2; no longer C47.2, C48.2
- net GND: now also C47.2, C48.2, C50.1, C51.1
- net INPUT_IMPEDANCE: now reaches C40.2, C49.2, R40.1, U40.3 (+)
