File: Rev_1/ECAD/main_board/equalizer_channel_b.kicad_sch (KiCad schematic)
At the start: 27 parts, among them U40 NE5532, U41 NE5532

Commit message: Probably finished with PCB
Parts:
- removed U40, U41: NE5532, Package_SO:SOIC-8_3.9x4.9mm_P1.27mm, symbol Amplifier_Operational:NE5532
- added TP14: FILTER 1, TestPoint:TestPoint_Pad_1.0x1.0mm, symbol Connector:TestPoint
- added TP15: FILTER 2, TestPoint:TestPoint_Pad_1.0x1.0mm, symbol Connector:TestPoint
- added U8, U9: OPA1652, Package_SO:JEITA_SOIC-8_3.9x4.9mm_P1.27mm, symbol filip:OPA1652
- C32: renamed from C49; ID (none) -> 41
- C33: renamed from C47; ID (none) -> 25
- C34: renamed from C48; ID (none) -> 25
- C35: renamed from C50; ID (none) -> 25
- C36: renamed from C44; ID (none) -> 8
- C37: renamed from C45; ID (none) -> 8
- C38: renamed from C51; ID (none) -> 25
- C39: renamed from C46; ID (none) -> 8
- C40: renamed from C41; value 330n -> 27n
- C41: renamed from C42; ID (none) -> 39
- C42: renamed from C43; ID (none) -> 40
- R33: renamed from R40; ID (none) -> 44
- R34: renamed from R42; ID (none) -> 14
- R35: renamed from R43; ID (none) -> 67
- R36: renamed from R41; ID (none) -> 14
- R37: renamed from R44; ID (none) -> 67
- R38: renamed from R51; ID (none) -> 43
- R39: renamed from R45; ID (none) -> 66
- R40: renamed from R49; ID (none) -> 46
- R41: renamed from R50; ID (none) -> 67
- R42: renamed from R46; ID (none) -> 14
- R43: renamed from R47; ID (none) -> 47
- R44: renamed from R52; ID (none) -> 47
- R45: renamed from R48; ID (none) -> 45
- renumbered C40 to C31
Connections:
- net -5V is gone; now on net GND: C34.1, C38.2
- net GND: now also U8.4 (V-), U9.4 (V-); no longer C32.1, C33.2, C34.2, C35.1, C38.1, C42.1, R33.2, R35.2, R38.1
- net INPUT_IMPEDANCE: now also U8.3 (+)
- net OUT: now also TP15.1, U9.6 (-), U9.7
- net at R34.1, R36.1: now also U8.2 (-)
- net at C41.1, R43.2, R44.1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: now also TP14.1
- net at C37.2, R40.2, R44.2: now also U8.7
- net at C42.2, R45.2: now also U9.5 (+)
- net at C40.1, R39.2, R42.1: now also U9.2 (-)
- net at C40.2, R42.2, R43.1: now also U9.1
- net at C39.2, R41.1: now also U8.6 (-)
- net at C36.1, R36.2, R37.1: now also U8.1
- net +5V renamed +8V
- net +8V: now also U8.8 (V+), U9.8 (V+)
- new net +4V: C32.1, C33.2, C34.2, C35.1, C38.1, C42.1, R33.2, R35.2, R38.1, U8.5 (+), U9.3 (+)

Commit message: Exported Gerber and IBOM
Parts:
- TP14, TP15: now left out of the parts list
Changed lines of the file:
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@@
 		(body_style 1)
 		(exclude_from_sim no)
-		(in_bom yes)
+		(in_bom no)
 		(on_board yes)
 		(in_pos_files yes)
@@
 		(body_style 1)
 		(exclude_from_sim no)
-		(in_bom yes)
-		(on_board yes)
-		(in_pos_files yes)
+		(in_bom no)
+		(on_board yes)
+		(in_pos_files yes)

Commit message: Finished with adding 9V Power Delivery
Parts:
- C31: ID (none) -> 94
- C40: ID (none) -> 95
- U8, U9: ID (none) -> 100
Changed lines of the file:
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@@
 			)
 		)
-		(property "ID" ""
+		(property "ID" "94"
 			(at 49.53 86.36 90)
 			(hide yes)
@@
 			)
 		)
+		(property "ID" "100"
+			(at 88.9 88.9 0)
+			(hide yes)
+			(show_name no)
+			(do_not_autoplace no)
+			(effects
+				(font
+					(size 1.27 1.27)
+				)
+			)
+		)
 		(pin "6"
 		)
@@
 			)
 		)
+		(property "ID" "100"
+			(at 72.39 63.5 0)
+			(hide yes)
+			(show_name no)
+			(do_not_autoplace no)
+			(effects
+				(font
+					(size 1.27 1.27)
+				)
+			)
+		)
 		(pin "2"
 		)
@@
 			)
 		)
+		(property "ID" "100"
+			(at 147.32 91.44 0)
+			(hide yes)
+			(show_name no)
+			(do_not_autoplace no)
+			(effects
+				(font
+					(size 1.27 1.27)
+				)
+			)
+		)
 		(pin "5"
 		)
@@
 			)
 		)
-		(property "ID" ""
+		(property "ID" "95"
 			(at 147.32 67.31 90)
 			(hide yes)
@@
 			)
 		)
+		(property "ID" "100"
+			(at 204.47 88.9 0)
+			(hide yes)
+			(show_name no)
+			(do_not_autoplace no)
+			(effects
+				(font
+					(size 1.27 1.27)
+				)
+			)
+		)
 		(pin "8"
 		)
@@
 			)
 		)
+		(property "ID" "100"
+			(at 149.86 132.08 0)
+			(hide yes)
+			(show_name no)
+			(do_not_autoplace no)
+			(effects
+				(font
+					(size 1.27 1.27)
+				)
+			)
+		)
 		(pin "7"
 		)
@@
 			(at 109.22 63.5 0)
 			(hide yes)
+			(show_name no)
+			(do_not_autoplace no)
+			(effects
+				(font
+					(size 1.27 1.27)
+				)
+			)
+		)
+		(property "ID" "100"
+			(at 109.22 63.5 0)
+			(hide yes)
