File: Rev_1/ECAD/main_board/riaa_preamp.kicad_pcb (KiCad board)
At the start: 2 copper layers, 79 parts, among them J1 USB_C_Receptacle_PowerOnly_6P, U1 TPS60403DBV, U2 NE5532, U20 NE5532, U21 NE5532, U40 NE5532, U41 NE5532

Commit message: Finished
Parts:
- removed R40+1: 47k, Resistor_SMD:R_0805_2012Metric
- added C11: 100n, Capacitor_SMD:C_0805_2012Metric, F.Cu at (191.5, 100.4)
- added C12: 100n, Capacitor_SMD:C_0805_2012Metric, F.Cu at (157.6, 107.2)
- added C30: 100n, Capacitor_SMD:C_0805_2012Metric, F.Cu at (151.3, 78.5)
- added C31: 100n, Capacitor_SMD:C_0805_2012Metric, F.Cu at (144.5, 93.8)
- added C50: 100n, Capacitor_SMD:C_0805_2012Metric, F.Cu at (125.7, 85.9)
- added C51: 100n, Capacitor_SMD:C_0805_2012Metric, F.Cu at (122.2, 93.6)
- added D4: Yellow, LED_SMD:LED_0603_1608Metric_Pad1.05x0.95mm_HandSolder, F.Cu at (129.9, 110.4)
- added G***: LOGO, LOGO, F.Cu at (182.5, 120.0)
- added G***: LOGO, LOGO, F.Cu at (129.8, 118.4)
- added H1: Hole, MountingHole:MountingHole_2.7mm_M2.5_ISO14580_Pad, F.Cu at (112.0, 67.0)
- added H2: Hole, MountingHole:MountingHole_2.7mm_M2.5_ISO14580_Pad, F.Cu at (199.0, 67.0)
- added H3: Hole, MountingHole:MountingHole_2.7mm_M2.5_ISO14580_Pad, F.Cu at (199.0, 129.0)
- added H4: Hole, MountingHole:MountingHole_2.7mm_M2.5_ISO14580_Pad, F.Cu at (112.0, 129.0)
- added J2: RCJ-013, filip:RCJ-013, F.Cu at (145.0, 64.5)
- added J3: RCJ-013, filip:RCJ-013, F.Cu at (185.0, 64.5)
- added J4: RCJ-013, filip:RCJ-013, F.Cu at (126.0, 64.5)
- added J5: RCJ-013, filip:RCJ-013, F.Cu at (166.0, 64.5)
- added R12: 5k1, Resistor_SMD:R_0805_2012Metric, F.Cu at (145.3, 109.2)
- added R13: 1k, Resistor_SMD:R_0805_2012Metric, F.Cu at (162.7, 112.8)
- added R14: 1k, Resistor_SMD:R_0805_2012Metric, F.Cu at (148.8, 112.0)
- added R40: 47k, Resistor_SMD:R_0805_2012Metric, F.Cu at (123.6, 76.2)
- added TP1: GND, TestPoint:TestPoint_THTPad_1.0x1.0mm_Drill0.5mm, F.Cu at (173.2, 91.2)
- added TP2: 5V, TestPoint:TestPoint_THTPad_1.0x1.0mm_Drill0.5mm, F.Cu at (173.2, 85.9)
- added TP3: -5V, TestPoint:TestPoint_THTPad_1.0x1.0mm_Drill0.5mm, F.Cu at (173.2, 96.5)
- C5: footprint Capacitor_THT:C_Radial_D10.0mm_H12.5mm_P5.00mm -> Capacitor_THT:C_Radial_D6.3mm_H11.0mm_P2.50mm
- C8, C9: value 1u -> 22n
- D1: footprint Diode_SMD:D_0805_2012Metric -> Diode_SMD:D_SOD-123
- D2, D3: footprint Diode_SMD:D_0805_2012Metric -> LED_SMD:LED_1206_3216Metric
- R10, R11: value 5k1 -> 1k
- R6: value 500 -> 1k
- R7: value 10k -> 1k
- R8: value 500 -> 330
- R9: value 10k -> 330
- RV1: value 1k -> 100k
- U2, U20, U21, U40, U41: footprint Package_SO:SOIC-8_5.3x6.2mm_P1.27mm -> Package_SO:SOIC-8_3.9x4.9mm_P1.27mm
- moved C1 277.3 mm to (200.2, 106.4), turned to -90 degrees
- moved C2 275.6 mm to (198.4, 109.5)
- moved C3 270.2 mm to (194.5, 106.6), turned to 90 degrees
- moved C4 267.4 mm to (192.4, 106.6), turned to 90 degrees
- moved D1 264.3 mm to (193.9, 101.1), turned to 90 degrees
- moved C6 261.9 mm to (189.5, 98.3), turned to 90 degrees
- moved R2 259.6 mm to (193.9, 94.7), turned to 90 degrees
- moved C7 258.2 mm to (186.7, 97.2)
- moved R3 257.0 mm to (191.8, 94.7), turned to 90 degrees
- moved U1 253.9 mm to (197.4, 106.4), turned to 90 degrees
- moved FB1 250.8 mm to (186.7, 99.2), turned to 180 degrees
- moved R1 245.9 mm to (193.8, 109.6), turned to 180 degrees
- moved C5 244.3 mm to (187.5, 102.4), turned to -90 degrees
- moved J1 241.5 mm to (199.5, 98.0), turned to 90 degrees
- moved C8 235.1 mm to (160.7, 109.2), turned to 90 degrees
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Connections:
- net Net-(U1-C_{FLY+}) renamed /CFLY+
- net Net-(U1-C_{FLY-}) renamed /CFLY-
- net Net-(U1-OUT) renamed /UNFILTERED_-5V
- net Net-(U20A-+) renamed /Equalizer Channel A/INPUT_IMPEDANCE
- net Net-(U2A--) renamed /R_INV
- net Net-(U40A-+) renamed /Equalizer Channel B/INPUT_IMPEDANCE
- C20 pad 1: /Equalizer Channel A/IN -> /RIGHT_CHANNEL_IN
- C22 pad 2: /Equalizer Channel A/OUT -> /RIGHT_CHANNEL_EQUALIZED
- C27 pad 2: -5V -> GND
- C28 pad 1: +5V -> GND
- C28 pad 2: -5V -> +5V
- C40 pad 1: /Equalizer Channel B/IN -> /LEFT_CHANNEL_IN
- C42 pad 2: /Equalizer Channel B/OUT -> /LEFT_CHANNEL_EQUALIZED
- C47 pad 2: -5V -> GND
- C48 pad 1: +5V -> -5V
- C48 pad 2: -5V -> GND
- C8 pad 1: Net-(C8-Pad1) -> /R_CHANNEL_HP
- C9 pad 1: Net-(C9-Pad1) -> /L_CHANNEL_HP
- D2 pad 1: Net-(D2-K) -> GND
- D2 pad 2: GND -> /5V_LED
- D3 pad 1: GND -> /-5V_LED
- D3 pad 2: Net-(D3-A) -> GND
- R10 pad 1: Net-(R10-Pad1) -> /L_INV
- R10 pad 2: Net-(C8-Pad1) -> /L_POT_OUT
- R11 pad 1: Net-(R11-Pad1) -> GND
- R11 pad 2: Net-(C9-Pad1) -> /L_INV
- R4 pad 2: Net-(D2-K) -> /5V_LED
- R5 pad 2: Net-(D3-A) -> /-5V_LED
- R6 pad 2: Net-(R6-Pad2) -> /R_POT_OUT
- R8 pad 1: Net-(U2B--) -> /RIGHT_CHANNEL_EQUALIZED
- R8 pad 2: Net-(R8-Pad2) -> /R_CHANNEL_HP
- R9 pad 1: GND -> /LEFT_CHANNEL_EQUALIZED
- R9 pad 2: Net-(U2B--) -> /L_CHANNEL_HP
- RV1 pad 1: Net-(R6-Pad2) -> /R_POT_OUT
- RV1 pad 2: Net-(R10-Pad1) -> /RIGHT_CHANNEL_OUT
- RV1 pad 3: GND -> /RIGHT_CHANNEL_OUT
- RV1 pad 4: Net-(R8-Pad2) -> /L_POT_OUT
- RV1 pad 5: Net-(R11-Pad1) -> /LEFT_CHANNEL_OUT
- RV1 pad 6: GND -> /LEFT_CHANNEL_OUT
- U2 pad 1: Net-(R6-Pad2) -> /RIGHT_CHANNEL_OUT
- U2 pad 3: /Equalizer Channel A/OUT -> /R_CHANNEL_HP
- U2 pad 4: GND -> -5V
- U2 pad 5: /Equalizer Channel B/OUT -> /L_CHANNEL_HP
- U2 pad 6: Net-(U2B--) -> /L_INV
- U2 pad 7: Net-(R8-Pad2) -> /LEFT_CHANNEL_OUT
- U21 pad 1: /Equalizer Channel A/OUT -> /RIGHT_CHANNEL_EQUALIZED
- U21 pad 2: /Equalizer Channel A/OUT -> /RIGHT_CHANNEL_EQUALIZED
- U41 pad 1: /Equalizer Channel B/OUT -> /LEFT_CHANNEL_EQUALIZED
- U41 pad 2: /Equalizer Channel B/OUT -> /LEFT_CHANNEL_EQUALIZED
Routing:
- net +5V: track 0.00 -> 197.6 mm, vias 0 -> 10
- net -5V: track 0.00 -> 188.3 mm, vias 0 -> 11
- net /RIGHT_CHANNEL_OUT: track 0.00 -> 102.3 mm, vias 0 -> 6
- net /LEFT_CHANNEL_OUT: track 0.00 -> 79.9 mm, vias 0 -> 6
- net GND: track 0.00 -> 48.6 mm, vias 0 -> 43
- net /LEFT_CHANNEL_EQUALIZED: track 0.00 -> 48.5 mm
- net /RIGHT_CHANNEL_EQUALIZED: track 0.00 -> 42.1 mm
- net /R_POT_OUT: track 0.00 -> 34.7 mm
- net /RIGHT_CHANNEL_IN: track 0.00 -> 20.2 mm
- net /LEFT_CHANNEL_IN: track 0.00 -> 19.9 mm
- net VBUS: track 0.00 -> 16.8 mm
- net /SUN_LED: track 0.00 -> 14.7 mm
- net Net-(C44-Pad1): track 0.00 -> 14.1 mm
- net Net-(C24-Pad1): track 0.00 -> 14.0 mm
- net Net-(C45-Pad2): track 0.00 -> 13.9 mm
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- added copper zone on F.Cu, net /UNFILTERED_-5V
- added copper zone on B.Cu, net GND
Other:
- board outline added: 95 x 70 mm
- board text added: "-5V"
- board text added: "5V"
- board text added: "GND"
- board text added: "LEFT IN"
- board text added: "LEFT OUT"
- board text added: "RIAA PREAMP"
- board text added: "RIGHT IN"
- board text added: "RIGHT OUT"
- board text added: "VOLUME"
