File: Rev_1/ECAD/main_board/riaa_preamp.kicad_pcb (KiCad board)
At the start: 2 copper layers, 95 x 70 mm, 102 parts, among them J1 USB_C_Receptacle_PowerOnly_6P, J2 RCJ-013, J3 RCJ-013, J4 RCJ-013, J5 RCJ-013, U1 TPS60403DBV, U2 NE5532, U20 NE5532, U21 NE5532, U40 NE5532, U41 NE5532

Commit message: Probably finished with PCB
Parts:
- removed C44, C45, C46: 22n, Capacitor_SMD:C_0805_2012Metric
- removed C47, C48, C50, C51: 100n, Capacitor_SMD:C_0805_2012Metric
- removed C49: 100p, Capacitor_SMD:C_0805_2012Metric
- removed the J1 at (199.5, 98.0)
- removed R49: 82k, Resistor_SMD:R_0805_2012Metric
- removed R50: 10k, Resistor_SMD:R_0805_2012Metric
- removed R51: 22k, Resistor_SMD:R_0805_2012Metric
- removed R52: 220k, Resistor_SMD:R_0805_2012Metric
- removed TP1: GND, TestPoint:TestPoint_THTPad_1.0x1.0mm_Drill0.5mm
- removed TP2: 5V, TestPoint:TestPoint_THTPad_1.0x1.0mm_Drill0.5mm
- removed U20, U21, U40, U41: NE5532, Package_SO:SOIC-8_3.9x4.9mm_P1.27mm
- added C13: 4u7, Capacitor_SMD:C_0805_2012Metric, F.Cu at (185.0, 108.3)
- added C14: 100n, Capacitor_SMD:C_0805_2012Metric, F.Cu at (153.7, 116.5)
- added C15: 100n, Capacitor_SMD:C_0805_2012Metric, F.Cu at (186.9, 110.4)
- added C16: 100n, Capacitor_SMD:C_0805_2012Metric, F.Cu at (157.4, 109.3)
- added C17: 10n, Capacitor_SMD:C_0603_1608Metric, F.Cu at (186.9, 116.3)
- added C18: 100n, Capacitor_SMD:C_0805_2012Metric, F.Cu at (176.1, 122.0)
- added C19: 330n, Capacitor_SMD:C_0805_2012Metric, F.Cu at (131.1, 73.7)
- added C32: 100p, Capacitor_SMD:C_0805_2012Metric, F.Cu at (150.4, 77.7)
- added C33: 100n, Capacitor_SMD:C_0805_2012Metric, F.Cu at (142.2, 82.9)
- added C34: 100n, Capacitor_SMD:C_0805_2012Metric, F.Cu at (146.7, 75.6)
- added C35: 100n, Capacitor_SMD:C_0805_2012Metric, F.Cu at (150.6, 84.6)
- added C36: 22n, Capacitor_SMD:C_0805_2012Metric, F.Cu at (143.3, 75.6)
- added C37: 22n, Capacitor_SMD:C_0805_2012Metric, F.Cu at (136.3, 79.5)
- added C38: 100n, Capacitor_SMD:C_0805_2012Metric, F.Cu at (139.3, 89.8)
- added C39: 22n, Capacitor_SMD:C_0805_2012Metric, F.Cu at (139.0, 78.6)
- added J3: USB_C_Receptacle_PowerOnly_6P, Connector_USB:USB_C_Receptacle_GCT_USB4125-xx-x-0190_6P_TopMnt_Horizontal, F.Cu at (199.7, 98.0)
- added R15: 22k, Resistor_SMD:R_0805_2012Metric, F.Cu at (166.9, 77.3)
- added R16: 22k, Resistor_SMD:R_0805_2012Metric, F.Cu at (185.8, 77.5)
- added R17: 10k, Resistor_SMD:R_0603_1608Metric, F.Cu at (191.8, 102.5)
- added R18: 22, Resistor_SMD:R_0603_1608Metric, F.Cu at (188.3, 108.2)
- added R19: 100k, Resistor_SMD:R_0805_2012Metric, F.Cu at (186.9, 118.1)
- added R33: 47k, Resistor_SMD:R_0805_2012Metric, F.Cu at (150.4, 75.7)
- added R34: 100k, Resistor_SMD:R_0805_2012Metric, F.Cu at (151.4, 80.4)
- added R35: 10k, Resistor_SMD:R_0805_2012Metric, F.Cu at (153.3, 78.9)
- added R36: 100k, Resistor_SMD:R_0805_2012Metric, F.Cu at (149.5, 80.4)
- added R37: 10k, Resistor_SMD:R_0805_2012Metric, F.Cu at (147.5, 83.2)
- added R38: 22k, Resistor_SMD:R_0805_2012Metric, F.Cu at (138.9, 76.6)
- added R39: 1k, Resistor_SMD:R_0805_2012Metric, F.Cu at (138.8, 84.3)
- added TP11: FILTER 1, TestPoint:TestPoint_Pad_1.0x1.0mm, F.Cu at (128.0, 91.2)
- added TP12: FILTER 2, TestPoint:TestPoint_Pad_1.0x1.0mm, F.Cu at (130.0, 86.9)
- added TP14: FILTER 1, TestPoint:TestPoint_Pad_1.0x1.0mm, F.Cu at (147.3, 91.2)
- added TP15: FILTER 2, TestPoint:TestPoint_Pad_1.0x1.0mm, F.Cu at (149.4, 86.9)
- added TP4: VOUT OFFSET, TestPoint:TestPoint_Pad_1.0x1.0mm, F.Cu at (184.9, 82.9)
- added TP5: VOUT, TestPoint:TestPoint_Pad_1.0x1.0mm, F.Cu at (166.0, 75.3)
- added TP6: VOUT, TestPoint:TestPoint_Pad_1.0x1.0mm, F.Cu at (185.0, 75.4)
- added TP7: GND, TestPoint:TestPoint_THTPad_1.0x1.0mm_Drill0.5mm, F.Cu at (190.0, 119.6)
- added TP8: 8V, TestPoint:TestPoint_THTPad_1.0x1.0mm_Drill0.5mm, F.Cu at (194.1, 119.6)
- added TP9: 4V, TestPoint:TestPoint_THTPad_1.0x1.0mm_Drill0.5mm, F.Cu at (197.9, 119.6)
- added U3: TPS72201, Package_TO_SOT_SMD:SOT-23-5, F.Cu at (186.9, 113.4)
- added U4: TLE2426xD, Package_SO:SOIC-8_3.9x4.9mm_P1.27mm, F.Cu at (181.0, 121.3)
- added U5: OPA1652, Package_SO:JEITA_SOIC-8_3.9x4.9mm_P1.27mm, F.Cu at (125.5, 79.2)
- added U6: OPA1652, Package_SO:JEITA_SOIC-8_3.9x4.9mm_P1.27mm, F.Cu at (125.5, 87.4)
- added U8: OPA1652, Package_SO:JEITA_SOIC-8_3.9x4.9mm_P1.27mm, F.Cu at (144.8, 79.2)
- added U9: OPA1652, Package_SO:JEITA_SOIC-8_3.9x4.9mm_P1.27mm, F.Cu at (144.8, 87.4)
- C1, C2: value 1u -> 330p
- C10: value 100n -> 1u
- C11, C6: value 100n -> 4u7
- C12: value 100n -> 47u; footprint Capacitor_SMD:C_0805_2012Metric -> Capacitor_THT:C_Radial_D6.3mm_H11.0mm_P2.50mm
- C20: value 330n -> 100p
- C21: value 330n -> 100n
- C22: value 470p -> 100n
- C23: value 330p -> 100n
- C25: value 22n -> 100n
- C27, C7: value 100n -> 22n
- C28: value 100n -> 27n
- C29: value 100p -> 470p
- C3: value 1u -> 100n
- C30: value 100n -> 330p
- C31: value 100n -> 330n
- C40: value 330n -> 27n
- C41: value 330n -> 470p
- C42: value 470p -> 330p
- C43: value 330p -> 10u
- C5: value 47u -> 10u; footprint Capacitor_THT:C_Radial_D6.3mm_H11.0mm_P2.50mm -> Capacitor_SMD:C_0805_2012Metric
- C9: value 22n -> 1u
- D1: value D_TVS -> TVS
- D2: value GREEN -> D_Schottky; footprint LED_SMD:LED_1206_3216Metric -> Diode_SMD:D_SOD-123
- D4: value Yellow -> GREEN; footprint LED_SMD:LED_0603_1608Metric_Pad1.05x0.95mm_HandSolder -> LED_SMD:LED_1206_3216Metric
- R1: value 50 -> 330; footprint Resistor_SMD:R_1206_3216Metric -> Resistor_SMD:R_0805_2012Metric
- R12: value 5k1 -> 1k
- R13, R14: value 1k -> 10k; footprint Resistor_SMD:R_0805_2012Metric -> Resistor_SMD:R_0603_1608Metric
- R2, R5: value 5k1 -> 191k; footprint Resistor_SMD:R_0805_2012Metric -> Resistor_SMD:R_0603_1608Metric
- R25: value 1k -> 22k
- R26: value 100k -> 1k
- R27: value 220k -> 82k
- R28: value 68k -> 10k
- R29: value 22k -> 100k
- R3: value 5k1 -> 9k5; footprint Resistor_SMD:R_0805_2012Metric -> Resistor_SMD:R_0603_1608Metric
- R30: value 82k -> 220k
- R31, R43, R44: value 10k -> 220k
- R32: value 220k -> 68k
- R4: value 5k1 -> 330
- R40: value 47k -> 82k
- R41: value 100k -> 10k
- R45: value 1k -> 68k
- R46: value 100k -> 560k; footprint Resistor_SMD:R_0805_2012Metric -> Resistor_SMD:R_0603_1608Metric
- R47: value 220k -> 10k; footprint Resistor_SMD:R_0805_2012Metric -> Resistor_SMD:R_0603_1608Metric
- R48: value 68k -> 10k; footprint Resistor_SMD:R_0805_2012Metric -> Resistor_SMD:R_0603_1608Metric
- R6: value 1k -> 9k5; footprint Resistor_SMD:R_0805_2012Metric -> Resistor_SMD:R_0603_1608Metric
- R8, R9: value 330 -> 1k
- TP3: value -5V -> VOUT OFFSET; footprint TestPoint:TestPoint_THTPad_1.0x1.0mm_Drill0.5mm -> TestPoint:TestPoint_Pad_1.0x1.0mm
- U1: value TPS60403DBV -> OPA1652; footprint Package_TO_SOT_SMD:SOT-23-5 -> Package_SO:JEITA_SOIC-8_3.9x4.9mm_P1.27mm
- U2: value NE5532 -> TPS25730D; footprint Package_SO:SOIC-8_3.9x4.9mm_P1.27mm -> Package_DFN_QFN:Texas_REF0038A_WQFN-38-2EP_6x4mm_P0.4
- moved C43 74.0 mm to (189.6, 113.7)
- moved G*** 73.2 mm to (195.0, 85.0)
- moved R46 72.9 mm to (184.3, 115.6), turned to 90 degrees
- moved D3 68.1 mm to (179.0, 88.0), turned to -90 degrees
- moved R47 62.4 mm to (179.0, 91.8), turned to 90 degrees
- moved R5 60.6 mm to (178.1, 103.4), turned to -90 degrees
- moved R48 59.4 mm to (175.6, 92.0), turned to 90 degrees
- moved D2 57.8 mm to (184.7, 100.4)
- moved G*** 55.7 mm to (127.5, 111.5)
- moved D4 50.9 mm to (175.6, 88.0), turned to -90 degrees
- moved C10 47.5 mm to (184.9, 80.1), turned to 90 degrees
- moved R1 45.5 mm to (148.3, 111.3), turned to 0 degrees
- moved R14 44.3 mm to (191.8, 101.1), turned to 0 degrees
- moved U1 42.2 mm to (155.7, 113.0), turned to 180 degrees
- moved R31 39.1 mm to (116.8, 82.9)
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- renumbered J4 to J1, J5 to J4, J3 to J5
Connections:
- C1 pad 1: /CFLY+ -> /CC2
- C1 pad 2: /CFLY- -> GND
- C10 pad 1: +5V -> /LEFT_CHANNEL_OUT
- C10 pad 2: GND -> Net-(C10-Pad2)
- C11 pad 1: VBUS -> /LDO_1V5
- C12 pad 1: -5V -> +9V
- C2 pad 1: +5V -> /CC1
- C20 pad 1: /RIGHT_CHANNEL_IN -> +4V
- C21 pad 1: Net-(U20B--) -> +8V
- C21 pad 2: Net-(C21-Pad2) -> +4V
- C22 pad 1: Net-(C22-Pad1) -> GND
- C22 pad 2: /RIGHT_CHANNEL_EQUALIZED -> +4V
- C23 pad 1: GND -> +4V
- C23 pad 2: Net-(U21A-+) -> +8V
- C25 pad 1: Net-(C24-Pad2) -> +4V
- C25 pad 2: Net-(C25-Pad2) -> GND
- C26 pad 2: Net-(U21B--) -> Net-(C26-Pad2)
- C27 pad 1: +5V -> Net-(C24-Pad2)
- C27 pad 2: GND -> Net-(U5B--)
- C28 pad 1: GND -> Net-(U6A--)
- C28 pad 2: +5V -> Net-(C28-Pad2)
- C29 pad 1: GND -> Net-(C29-Pad1)
- C29 pad 2: /Equalizer Channel A/INPUT_IMPEDANCE -> /RIGHT_CHANNEL_EQUALIZED
- C3 pad 1: /UNFILTERED_-5V -> VBUS
- C30 pad 1: -5V -> +4V
- C30 pad 2: GND -> Net-(U6B-+)
- C31 pad 1: GND -> /LEFT_CHANNEL_IN
- C31 pad 2: -5V -> /Equalizer Channel B/INPUT_IMPEDANCE
- C4 pad 1: -5V -> Net-(D2-K)
- C40 pad 1: /LEFT_CHANNEL_IN -> Net-(U9A--)
- C40 pad 2: /Equalizer Channel B/INPUT_IMPEDANCE -> Net-(C40-Pad2)
- C41 pad 1: Net-(U40B--) -> Net-(C41-Pad1)
- C41 pad 2: Net-(C41-Pad2) -> /LEFT_CHANNEL_EQUALIZED
- C42 pad 1: Net-(C42-Pad1) -> +4V
- C42 pad 2: /LEFT_CHANNEL_EQUALIZED -> Net-(U9B-+)
- C43 pad 1: GND -> +8V
- C43 pad 2: Net-(U41A-+) -> GND
- C5 pad 1: VBUS -> /LDO_3V3
- C6 pad 1: VBUS -> Net-(D2-K)
- C7 pad 1: +5V -> /L_CHANNEL_HP
- C7 pad 2: GND -> +4V
- C8 pad 2: GND -> +4V
- C9 pad 1: /L_CHANNEL_HP -> /RIGHT_CHANNEL_OUT
- C9 pad 2: GND -> Net-(C9-Pad2)
- D1 pad 1: GND -> VBUS
- D1 pad 2: VBUS -> GND
- D2 pad 1: GND -> Net-(D2-K)
- D2 pad 2: /5V_LED -> GND
- D3 pad 1: /-5V_LED -> GND
- D3 pad 2: GND -> Net-(D3-A)
- D4 pad 2: /SUN_LED -> Net-(D4-A)
- FB1 pad 2: +5V -> Net-(D2-K)
- J1 pad 1A: /LEFT_CHANNEL_IN -> GND
- J1 pad 1B: /LEFT_CHANNEL_IN -> GND
- J1 pad 1C: /LEFT_CHANNEL_IN -> GND
- J1 pad 2: GND -> /RIGHT_CHANNEL_IN
- J2 pad 1A: /RIGHT_CHANNEL_IN -> GND
- J2 pad 1B: /RIGHT_CHANNEL_IN -> GND
- J2 pad 1C: /RIGHT_CHANNEL_IN -> GND
- J2 pad 2: GND -> /LEFT_CHANNEL_IN
- J4 pad 1A: /LEFT_CHANNEL_OUT -> GND
- J4 pad 1B: /LEFT_CHANNEL_OUT -> GND
- J4 pad 1C: /LEFT_CHANNEL_OUT -> GND
- J4 pad 2: GND -> Net-(C9-Pad2)
- J5 pad 1A: /RIGHT_CHANNEL_OUT -> GND
- J5 pad 1B: /RIGHT_CHANNEL_OUT -> GND
- J5 pad 1C: /RIGHT_CHANNEL_OUT -> GND
- J5 pad 2: GND -> Net-(C10-Pad2)
- R1 pad 1: /UNFILTERED_-5V -> /LEFT_CHANNEL_EQUALIZED
- R1 pad 2: -5V -> /L_CHANNEL_HP
- R10 pad 1: /L_INV -> +4V
- R10 pad 2: /L_POT_OUT -> /L_INV
- R11 pad 1: GND -> /R_INV
- R11 pad 2: /L_INV -> /R_POT_OUT
- R12 pad 1: +5V -> /L_INV
- R12 pad 2: /SUN_LED -> /L_POT_OUT
- R13 pad 1: GND -> Net-(R13-Pad1)
- R13 pad 2: /R_INV -> GND
- R14 pad 1: GND -> Net-(R14-Pad1)
- R14 pad 2: /L_INV -> GND
- R2 pad 1: Net-(J1-CC2) -> /LDO_3V3
- R2 pad 2: GND -> Net-(U2-ADCIN2)
- R20 pad 2: GND -> +4V
- R22 pad 2: GND -> +4V
- R25 pad 1: Net-(R24-Pad2) -> +4V
- R25 pad 2: Net-(U20B--) -> Net-(C24-Pad2)
- R26 pad 1: Net-(U20B--) -> Net-(R24-Pad2)
- R26 pad 2: Net-(C21-Pad2) -> Net-(U6A--)
- R27 pad 1: Net-(C21-Pad2) -> Net-(R27-Pad1)
- R27 pad 2: Net-(C22-Pad1) -> Net-(C26-Pad2)
- R28 pad 1: Net-(C22-Pad1) -> Net-(U5B--)
- R28 pad 2: Net-(U21A-+) -> Net-(R27-Pad1)
- R29 pad 1: GND -> Net-(U6A--)
- R29 pad 2: Net-(C24-Pad2) -> Net-(C28-Pad2)
- R3 pad 1: Net-(J1-CC1) -> Net-(U2-ADCIN2)
- R30 pad 1: Net-(R30-Pad1) -> Net-(C28-Pad2)
- R30 pad 2: Net-(C25-Pad2) -> Net-(C29-Pad1)
- R31 pad 1: Net-(U21B--) -> Net-(C29-Pad1)
- R31 pad 2: Net-(R30-Pad1) -> Net-(C26-Pad2)
- R32 pad 1: Net-(C22-Pad1) -> Net-(C29-Pad1)
- R32 pad 2: Net-(C25-Pad2) -> Net-(U6B-+)
- R4 pad 1: +5V -> /RIGHT_CHANNEL_EQUALIZED
- R4 pad 2: /5V_LED -> /R_CHANNEL_HP
- R40 pad 1: /Equalizer Channel B/INPUT_IMPEDANCE -> Net-(R40-Pad1)
- R40 pad 2: GND -> Net-(C37-Pad2)
- R41 pad 1: Net-(U40A--) -> Net-(U8B--)
- R41 pad 2: Net-(C44-Pad1) -> Net-(R40-Pad1)
- R42 pad 1: Net-(U40A--) -> Net-(U9A--)
- R42 pad 2: Net-(R42-Pad2) -> Net-(C40-Pad2)
- R43 pad 1: Net-(R42-Pad2) -> Net-(C40-Pad2)
- R43 pad 2: GND -> Net-(C41-Pad1)
- R44 pad 1: Net-(C44-Pad1) -> Net-(C41-Pad1)
- R44 pad 2: Net-(R44-Pad2) -> Net-(C37-Pad2)
- R45 pad 1: Net-(R44-Pad2) -> Net-(C41-Pad1)
- R45 pad 2: Net-(U40B--) -> Net-(U9B-+)
- R46 pad 1: Net-(U40B--) -> /FB
- R46 pad 2: Net-(C41-Pad2) -> GND
- R47 pad 1: Net-(C41-Pad2) -> +8V
- R47 pad 2: Net-(C42-Pad1) -> Net-(D3-A)
- R48 pad 1: Net-(C42-Pad1) -> +4V
- R48 pad 2: Net-(U41A-+) -> Net-(D4-A)
- R5 pad 1: -5V -> /LDO_3V3
- R5 pad 2: /-5V_LED -> Net-(U2-ADCIN1)
- R6 pad 1: /R_INV -> Net-(U2-ADCIN1)
- R6 pad 2: /R_POT_OUT -> GND
- R7 pad 1: GND -> +4V
- R8 pad 1: /RIGHT_CHANNEL_EQUALIZED -> +4V
- R8 pad 2: /R_CHANNEL_HP -> /L_INV
- R9 pad 1: /LEFT_CHANNEL_EQUALIZED -> +4V
- R9 pad 2: /L_CHANNEL_HP -> /R_INV
- TP3 pad 1: -5V -> /RIGHT_CHANNEL_OUT
- U1 pad 1: /UNFILTERED_-5V -> /RIGHT_CHANNEL_OUT
- U1 pad 2: +5V -> /R_INV
- U1 pad 3: /CFLY- -> /R_CHANNEL_HP
- U1 pad 5: /CFLY+ -> /L_CHANNEL_HP
- U2 pad 1: /RIGHT_CHANNEL_OUT -> /LDO_3V3
- U2 pad 2: /R_INV -> Net-(U2-ADCIN1)
- U2 pad 3: /R_CHANNEL_HP -> Net-(U2-ADCIN2)
- U2 pad 4: -5V -> /LDO_1V5
- U2 pad 5: /L_CHANNEL_HP -> GND
- U2 pad 6: /L_INV -> /CAP_MIS
- U2 pad 7: /LEFT_CHANNEL_OUT -> GND
- U2 pad 8: +5V -> unconnected-(U2-I2Ct_SDA-Pad8)
Routing:
- net +5V: track 197.6 -> 0.00 mm, vias 10 -> 0
- net -5V: track 188.3 -> 0.00 mm, vias 11 -> 0
- net +8V: track 0.00 -> 162.5 mm, vias 0 -> 7
- net +4V: track 0.00 -> 119.1 mm, vias 0 -> 38
- net /RIGHT_CHANNEL_OUT: track 102.3 -> 65.9 mm, vias 6 -> 4
- net Net-(C41-Pad1): track 0.00 -> 30.0 mm
- net Net-(C29-Pad1): track 0.00 -> 29.1 mm
- net /RIGHT_CHANNEL_EQUALIZED: track 42.1 -> 67.7 mm, vias 0 -> 4
- net /LEFT_CHANNEL_EQUALIZED: track 48.5 -> 30.9 mm, vias 0 -> 2
- net /R_POT_OUT: track 34.7 -> 19.5 mm, vias 0 -> 2
- net /RIGHT_CHANNEL_IN: track 20.2 -> 5.44 mm
- net /SUN_LED: track 14.7 -> 0.00 mm
- net /LEFT_CHANNEL_IN: track 19.9 -> 5.74 mm
- net Net-(C44-Pad1): track 14.1 -> 0.00 mm
- net Net-(C45-Pad2): track 13.9 -> 0.00 mm
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- added copper zone on In2.Cu, net +4V
- added copper zone on In1.Cu, net GND
- removed copper zone on F.Cu, net /UNFILTERED_-5V
Other:
- copper layers 2 -> 4
- board text added: "+4V"
- board text added: "+8V"
- board text added: "GAIN"
- board text removed: "-5V"
- board text removed: "5V"
- board text removed: "VOLUME"

Commit message: Exported Gerber and IBOM
Parts:
- J3: footprint Connector_USB:USB_C_Receptacle_GCT_USB4125-xx-x-0190_6P_TopMnt_Horizontal -> Connector_USB:USB_C_Receptacle_GCT_USB4125-xx-x_6P_TopMnt_Horizontal
- R48: value 10k -> 3k3
Connections:
- J3 pad SH: (no net) -> GND
