File: Rev_1/ECAD/main_board/riaa_preamp.kicad_sch (KiCad schematic)
At the start: 15 parts, among them J1 USB_C_Receptacle_PowerOnly_6P, J2 RCJ-013, U2 TPS60403DBV

Commit message: Semi finsihed schematic
Parts:
- added C10: 100n, Capacitor_SMD:C_0805_2012Metric, symbol Device:C_Small
- added C8, C9: 1u, Capacitor_SMD:C_0805_2012Metric, symbol Device:C_Small
- added D2, D3: GREEN, Diode_SMD:D_0805_2012Metric, symbol Device:LED
- added J3, J4, J5: RCJ-013, filip:RCJ-013, symbol filip:RCJ-013
- added R10, R11, R4, R5: 5k1, Resistor_SMD:R_0805_2012Metric, symbol Device:R
- added R6, R8: 500, Resistor_SMD:R_0805_2012Metric, symbol Device:R
- added R7, R9: 10k, Resistor_SMD:R_0805_2012Metric, symbol Device:R
- added RV1: 1k, Potentiometer_THT:Potentiometer_Alps_RK163_Dual_Horizontal, symbol Device:R_Potentiometer_Dual_Separate
- added U2: NE5532, Package_SO:SOIC-8_5.3x6.2mm_P1.27mm, symbol Amplifier_Operational:NE5532
- C1, C2, C3, C4: footprint (none) -> Capacitor_SMD:C_0805_2012Metric
- C5: footprint (none) -> Capacitor_THT:C_Radial_D10.0mm_H12.5mm_P5.00mm
- D1: footprint (none) -> Diode_SMD:D_0805_2012Metric
- R1: footprint (none) -> Resistor_SMD:R_1206_3216Metric
- R2, R3: footprint (none) -> Resistor_SMD:R_0805_2012Metric
- renumbered U2 to U1
Connections:
- net +5V: now also C10.1, R4.1, U2.8 (V+)
- net -5V: now also R5.1
- net Equalizer Channel A/IN: now also J2.1A (1), J2.1B (1), J2.1C (1)
- net Equalizer Channel A/OUT: now also U2.3 (+)
- net Equalizer Channel B/IN: now also J4.1A (1), J4.1B (1), J4.1C (1)
- net Equalizer Channel B/OUT: now also U2.5 (+)
- net GND: now also J2.2, C10.2, C8.2, C9.2, D2.2 (A), D3.1 (K), J3.2, J4.2, J5.2, R7.1, R9.1, RV1.3, RV1.6, U2.4 (V-)
- new net: R8.2, RV1.4, U2.7
- new net: R11.1, RV1.5
- new net: C9.1, J5.1A (1), J5.1B (1), J5.1C (1), R11.2
- new net: R6.1, R7.2, U2.2 (-)
- new net: D2.1 (K), R4.2
- new net: R10.1, RV1.2
- new net: C8.1, J3.1A (1), J3.1B (1), J3.1C (1), R10.2
- new net: R8.1, R9.2, U2.6 (-)
- new net: D3.2 (A), R5.2
- new net: R6.2, RV1.1, U2.1
Other:
- moved on the sheet: J2

Commit message: Finished
Parts:
- removed R8: 500, Resistor_SMD:R_0805_2012Metric, symbol Device:R
- added C11: 100n, Capacitor_SMD:C_0805_2012Metric, symbol Device:C
- added C12: 100n, Capacitor_SMD:C_0805_2012Metric, symbol Device:C_Small
- added D4: Yellow, LED_SMD:LED_0603_1608Metric_Pad1.05x0.95mm_HandSolder, symbol Device:LED
- added H1, H2, H3, H4: Hole, MountingHole:MountingHole_2.7mm_M2.5_ISO14580_Pad, symbol Mechanical:MountingHole_Pad
- added R10, R13, R14: 1k, Resistor_SMD:R_0805_2012Metric, symbol Device:R
- added R12: 5k1, Resistor_SMD:R_0805_2012Metric, symbol Device:R
- added TP1: GND, TestPoint:TestPoint_THTPad_1.0x1.0mm_Drill0.5mm, symbol Connector:TestPoint
- added TP2: 5V, TestPoint:TestPoint_THTPad_1.0x1.0mm_Drill0.5mm, symbol Connector:TestPoint
- added TP3: -5V, TestPoint:TestPoint_THTPad_1.0x1.0mm_Drill0.5mm, symbol Connector:TestPoint
- C5: footprint Capacitor_THT:C_Radial_D10.0mm_H12.5mm_P5.00mm -> Capacitor_THT:C_Radial_D6.3mm_H11.0mm_P2.50mm
- C8, C9: value 1u -> 22n
- D1: footprint Diode_SMD:D_0805_2012Metric -> Diode_SMD:D_SOD-123
- D2, D3: footprint Diode_SMD:D_0805_2012Metric -> LED_SMD:LED_1206_3216Metric
- R11: value 5k1 -> 1k
- R6: value 500 -> 1k
- R7: value 10k -> 1k
- R8: renamed from R10; value 5k1 -> 330
- R9: value 10k -> 330
- RV1: value 1k -> 100k; footprint Potentiometer_THT:Potentiometer_Alps_RK163_Dual_Horizontal -> (none)
- RV1: value 1k -> 100k
- U2: footprint Package_SO:SOIC-8_5.3x6.2mm_P1.27mm -> Package_SO:SOIC-8_3.9x4.9mm_P1.27mm; Mouser No: (none) -> 595-NE5532DR
- U2: footprint (none) -> Package_SO:SOIC-8_3.9x4.9mm_P1.27mm; Mouser No: (none) -> 595-NE5532DR
Connections:
- net Equalizer Channel B/OUT is gone; now on net L_CHANNEL_HP: U2.5 (+)
- net +5V: now also R12.1, TP2.1
- net -5V: now also U2.4 (V-), C12.1, TP3.1
- net GND: now also D2.1 (K), D3.2 (A), R11.1, C11.2, C12.2, D4.1 (K), H1.1, H2.1, H3.1, H4.1, R13.1, R14.1, TP1.1; no longer D2.2 (A), D3.1 (K), R9.1, RV1.3, RV1.6, U2.4 (V-)
- net VBUS: now also C11.1
- net LEFT_CHANNEL_OUT: now reaches U2.7
- net LEFT_CHANNEL_OUT: now also J5.1A (1), J5.1B (1), J5.1C (1), RV1.5, RV1.6; no longer RV1.4
- net UNFILTERED_-5V: now reaches C3.1, R1.1, U1.1 (OUT)
- net CFLY-: now reaches C1.2, U1.3 (C_{FLY-})
- net CFLY+: now reaches C1.1, U1.5 (C_{FLY+})
- net R_INV: now reaches R6.1, R7.2, U2.2 (-)
- net R_INV: now also R13.2
- net 5V_LED: now reaches R4.2
- net 5V_LED: now also D2.2 (A); no longer D2.1 (K)
- net RIGHT_CHANNEL_EQUALIZED: now reaches R8.1
- net RIGHT_CHANNEL_EQUALIZED: no longer RV1.2
- net RIGHT_CHANNEL_OUT: now reaches J3.1A (1), J3.1B (1), J3.1C (1)
- net RIGHT_CHANNEL_OUT: now also RV1.2, RV1.3, U2.1; no longer C8.1, R8.2
- net L_CHANNEL_HP: now reaches R9.2
- net L_CHANNEL_HP: now also C9.1; no longer U2.6 (-)
- net -5V_LED: now reaches R5.2
- net -5V_LED: now also D3.1 (K); no longer D3.2 (A)
- net R_POT_OUT: now reaches R6.2, RV1.1
- net R_POT_OUT: no longer U2.1
- net Equalizer Channel A/IN renamed RIGHT_CHANNEL_IN
- net Equalizer Channel A/OUT renamed R_CHANNEL_HP
- net R_CHANNEL_HP: now also C8.1, R8.2
- net Equalizer Channel B/IN renamed LEFT_CHANNEL_IN
- new net LEFT_CHANNEL_EQUALIZED: R9.1
- new net L_INV: R10.1, R11.2, R14.2, U2.6 (-)
- new net L_POT_OUT: R10.2, RV1.4
- new net SUN_LED: D4.2 (A), R12.2
Other:
- note added: "FC: 22kHz Gain: 10dB - 46dB"
- moved on the sheet: C1, C10, C2, C3, C4, C5, C6, C7, C8, D1, D2, D3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
