File: Rev_1/ECAD/main_board/riaa_preamp.kicad_sch (KiCad schematic)
At the start: 46 parts, among them J1 USB_C_Receptacle_PowerOnly_6P, J2 RCJ-013, J3 RCJ-013, J4 RCJ-013, J5 RCJ-013, U1 TPS60403DBV, U2 NE5532

Commit message: Probably finished with PCB
Parts:
- removed C11: 100n, Capacitor_SMD:C_0805_2012Metric, symbol Device:C
- removed C5: 47u, Capacitor_THT:C_Radial_D6.3mm_H11.0mm_P2.50mm, symbol Device:C
- removed C7: 100n, Capacitor_SMD:C_0805_2012Metric, symbol Device:C_Small
- removed D1: D_TVS, Diode_SMD:D_SOD-123, symbol Device:D_TVS
- removed D2: GREEN, LED_SMD:LED_1206_3216Metric, symbol Device:LED
- removed R1: 50, Resistor_SMD:R_1206_3216Metric, symbol Device:R
- removed R12, R2, R3, R4, R5: 5k1, Resistor_SMD:R_0805_2012Metric, symbol Device:R
- removed U1: TPS60403DBV, Package_TO_SOT_SMD:SOT-23-5, symbol Regulator_SwitchedCapacitor:TPS60403DBV
- removed U2: NE5532, Package_SO:SOIC-8_3.9x4.9mm_P1.27mm, symbol Amplifier_Operational:NE5532
- added C10, C9: 1u, Capacitor_SMD:C_0805_2012Metric, symbol Device:C_Small
- added C11, C13: 4u7, Capacitor_SMD:C_0805_2012Metric, symbol Device:C_Small
- added C12: 47u, Capacitor_THT:C_Radial_D6.3mm_H11.0mm_P2.50mm, symbol Device:C_Polarized_Small
- added C15, C18: 100n, Capacitor_SMD:C_0805_2012Metric, symbol Device:C_Small
- added C17: 10n, Capacitor_SMD:C_0603_1608Metric, symbol Device:C_Small
- added C43, C5: 10u, Capacitor_SMD:C_0805_2012Metric, symbol Device:C_Small
- added D1: TVS, Diode_SMD:D_SOD-123, symbol Device:D_Zener
- added D2: D_Schottky, Diode_SMD:D_SOD-123, symbol Device:D_Schottky
- added R13, R14, R17, R47: 10k, Resistor_SMD:R_0603_1608Metric, symbol Device:R_Small
- added R15, R16: 22k, Resistor_SMD:R_0805_2012Metric, symbol Device:R
- added R18: 22, Resistor_SMD:R_0603_1608Metric, symbol Device:R_Small
- added R19: 100k, Resistor_SMD:R_0805_2012Metric, symbol Device:R_Small
- added R2, R5: 191k, Resistor_SMD:R_0603_1608Metric, symbol Device:R_Small
- added R3, R6: 9k5, Resistor_SMD:R_0603_1608Metric, symbol Device:R_Small
- added R46: 560k, Resistor_SMD:R_0603_1608Metric, symbol Device:R_Small
- added R48: 3k3, Resistor_SMD:R_0603_1608Metric, symbol Device:R_Small
- added TP3, TP4: VOUT OFFSET, TestPoint:TestPoint_Pad_1.0x1.0mm, symbol Connector:TestPoint
- added TP5, TP6: VOUT, TestPoint:TestPoint_Pad_1.0x1.0mm, symbol Connector:TestPoint
- added U1: OPA1652, Package_SO:JEITA_SOIC-8_3.9x4.9mm_P1.27mm, symbol filip:OPA1652
- added U2: TPS25730D, Package_DFN_QFN:Texas_REF0038A_WQFN-38-2EP_6x4mm_P0.4, symbol Interface_USB:TPS25730D
- added U3: TPS72201, Package_TO_SOT_SMD:SOT-23-5, symbol Regulator_Linear:TPS72201
- added U4: TLE2426xD, Package_SO:SOIC-8_3.9x4.9mm_P1.27mm, symbol Reference_Voltage:TLE2426xD
- C1, C2: value 1u -> 330p; ID (none) -> 40
- C14: renamed from C10; ID (none) -> 25
- C16: renamed from C12; ID (none) -> 25
- C3: value 1u -> 100n; ID (none) -> 25
- C4: ID (none) -> 25
- C6: value 100n -> 4u7; ID (none) -> 26
- C7: renamed from C9; ID (none) -> 8
- C8: ID (none) -> 8
- D4: value Yellow -> GREEN; footprint LED_SMD:LED_0603_1608Metric_Pad1.05x0.95mm_HandSolder -> LED_SMD:LED_1206_3216Metric
- FB1: ID (none) -> 51
- J3: renamed from J1; ID (none) -> 30
- R1: renamed from R9; ID (none) -> 68
- R10: renamed from R14; ID (none) -> 66
- R11: renamed from R6; ID (none) -> 66
- R12: renamed from R10; ID (none) -> 66
- R4: renamed from R8; ID (none) -> 68
- R7: ID (none) -> 66
- R8: renamed from R11; ID (none) -> 66
- R9: renamed from R13; ID (none) -> 66
- TP8: renamed from TP2; value 5V -> 8V
- TP9: renamed from TP3; value -5V -> 4V
- renumbered J4 to J1, J5 to J4, J3 to J5, TP1 to TP7
Connections:
- net -5V_LED is gone; now on net GND: D3.1 (K)
- net CFLY+ is gone; now on net CC2: C1.1
- net CFLY- is gone; now on net GND: C1.2
- net UNFILTERED_-5V is gone; now on net VBUS: C3.1
- net GND: now also C16.1, J1.1A (1), J1.1B (1), J1.1C (1), J2.1A (1), J2.1B (1), J2.1C (1), J4.1A (1), J4.1B (1), J4.1C (1), J5.1A (1), J5.1B (1), J5.1C (1), C11.2, C12.2, C13.2, C15.2, C18.2, C43.2, C5.2, D1.2 (A), D2.2 (A), R13.2, R14.2, R15.2, R16.2, R17.2, R3.2, R46.2, R6.2, U1.4 (V-), U2.11 (GND), U2.12 (GND), U2.14 (GND), U2.16 (GND), U2.17 (GND), U2.31 (GND), U2.34 (GND), U2.39 (GND), U2.5 (ADCIN3), U2.7 (ADCIN4), U3.2 (GND), U4.2 (COMMON); no longer C14.2, C16.2, C7.2, C8.2, D3.2 (A), J1.2, J2.2, J4.2, J5.2, R10.1, R7.1, R8.1, R9.1
- net LEFT_CHANNEL_IN: now also J2.2; no longer J1.1A (1), J1.1B (1), J1.1C (1)
- net LEFT_CHANNEL_OUT: now also C10.1, TP4.1, U1.7; no longer J4.1A (1), J4.1B (1), J4.1C (1)
- net L_CHANNEL_HP: now also U1.5 (+)
- net L_INV: now also U1.6 (-)
- net RIGHT_CHANNEL_IN: now also J1.2; no longer J2.1A (1), J2.1B (1), J2.1C (1)
- net RIGHT_CHANNEL_OUT: now also C9.1, TP3.1, U1.1; no longer J5.1A (1), J5.1B (1), J5.1C (1)
- net R_CHANNEL_HP: now also U1.3 (+)
- net R_INV: now also U1.2 (-)
- net VBUS: now also D1.1 (K); no longer C6.1
- net CC2: now reaches J3.B5 (CC2)
- net CC2: now also U2.29 (CC2)
- net CC1: now reaches J3.A5 (CC1)
- net CC1: now also C2.1, U2.28 (CC1)
- net +5V renamed +8V
- net +8V: now also C17.1, C43.1, R19.1, R47.1, U1.8 (V+), U3.5 (VOUT), U4.3 (IN); no longer C2.1, FB1.2
- removed net -5V: C16.1, C4.1, TP9.1
- net SUN_LED: no longer names the net of D4.2 (A)
- net SUN_LED: now also R48.2
- new net: C13.1, C15.1, R18.2, U3.1 (VIN), U3.3 (EN)
- new net: R5.2, R6.1, U2.2 (ADCIN1)
- new net: C4.1, C6.1, D2.1 (K), FB1.2, U2.23 (VBUS_IN), U2.32 (VBUS)
- new net: R17.1, U2.26 (RESERVED)
- new net: R14.1, U2.27 (RESERVED)
- new net: R2.2, R3.1, U2.3 (ADCIN2)
- new net: R13.1, U2.36 (RESERVED)
- new net: C9.2, J4.2, R15.1, TP5.1
- new net: D3.2 (A), R47.2
- new net: C18.1, U4.8 (NOISE_REDUCTION)
- new net: C10.2, J5.2, R16.1, TP6.1
- new net +4V: C14.2, C16.2, C7.2, C8.2, R10.1, R48.1, R7.1, R8.1, R9.1, TP9.1, U4.1 (OUT)
- new net +9V: C12.1, R18.1, U2.20 (PPHV)
- new net CAP_MIS: U2.6 (CAP_MIS)
- new net FB: C17.2, R19.2, R46.1, U3.4 (FB)
- new net LDO_1V5: C11.1, U2.4 (LDO_1V5)
- new net LDO_3V3: C5.1, R2.1, R5.1, U2.1 (LDO_3V3)
- no-connect marks 0 -> 10
Other:
- note added: "TPS7E7101DBVR"
- note removed: "Calculate the maximum voltage drop across the resisor"
- note removed: "LOW ESR"
- moved on the sheet: C14, C16, C7, C8, J1, J2, J3, J4, J5, R1, R10, R11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

Commit message: Exported Gerber and IBOM
Parts:
- J3: footprint Connector_USB:USB_C_Receptacle_GCT_USB4125-xx-x-0190_6P_TopMnt_Horizontal -> Connector_USB:USB_C_Receptacle_GCT_USB4125-xx-x_6P_TopMnt_Horizontal; ID 30 -> (none)
- TP3, TP4, TP5, TP6, TP7, TP8, TP9: now left out of the parts list
Connections:
- net GND: now also J3.SH (SHIELD); no longer J3.S1 (SHIELD)
Changed lines of the file:
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@@
 	)
 	(symbol
+		(lib_name "USB_C_Receptacle_PowerOnly_6P_1")
+		(lib_id "Connector:USB_C_Receptacle_PowerOnly_6P")
+		(at 35.56 43.18 0)
+		(unit 1)
+		(body_style 1)
+		(exclude_from_sim no)
+		(in_bom yes)
+		(on_board yes)
+		(in_pos_files yes)
+		(dnp no)
+		(fields_autoplaced yes)
+		(property "Reference" "J3"
+			(at 35.56 25.4 0)
+			(show_name no)
+			(do_not_autoplace no)
+			(effects
+				(font
+					(size 1.27 1.27)
+				)
+			)
+		)
+		(property "Value" "USB_C_Receptacle_PowerOnly_6P"
+			(at 35.56 27.94 0)
+			(show_name no)
+			(do_not_autoplace no)
+			(effects
+				(font
+					(size 1.27 1.27)
+				)
+			)
+		)
+		(property "Footprint" "Connector_USB:USB_C_Receptacle_GCT_USB4125-xx-x_6P_TopMnt_Horizontal"
+			(at 39.37 40.64 0)
+			(hide yes)
+			(show_name no)
+			(do_not_autoplace no)
+			(effects
+				(font
+					(size 1.27 1.27)
+				)
+			)
+		)
+		(property "Datasheet" "https://www.usb.org/sites/default/files/documents/usb_type-c.zip"
+			(at 35.56 43.18 0)
+			(hide yes)
+			(show_name no)
+			(do_not_autoplace no)
+			(effects
+				(font
+					(size 1.27 1.27)
+				)
+			)
+		)
+		(property "Description" "USB Power-Only 6P Type-C Receptacle connector"
+			(at 35.56 43.18 0)
+			(hide yes)
+			(show_name no)
+			(do_not_autoplace no)
+			(effects
+				(font
+					(size 1.27 1.27)
+				)
+			)
+		)
+		(pin "A5"
+		)
+		(pin "A9"
+		)
+		(pin "B5"
+		)
+		(pin "B9"
+		)
+		(pin "B12"
+		)
+		(pin "SH"
+		)
+		(pin "A12"
+		)
+		(instances
+			(project "riaa_preamp"
+				(path "/2b990f77-15c8-4cc2-b07f-63b4e432ca20"
+					(reference "J3")
+					(unit 1)
+				)
+			)
+		)
+	)
+	(symbol
 		(lib_id "Device:R")
 		(at 118.11 177.8 180)
@@
 		(body_style 1)
 		(exclude_from_sim no)
-		(in_bom yes)
+		(in_bom no)
 		(on_board yes)
 		(in_pos_files yes)
@@
 		(body_style 1)
 		(exclude_from_sim no)
-		(in_bom yes)
+		(in_bom no)
 		(on_board yes)
 		(in_pos_files yes)
@@
 		(body_style 1)
 		(exclude_from_sim no)
-		(in_bom yes)
+		(in_bom no)
 		(on_board yes)
 		(in_pos_files yes)
@@
 		(body_style 1)
 		(exclude_from_sim no)
-		(in_bom yes)
+		(in_bom no)
 		(on_board yes)
 		(in_pos_files yes)
@@
 		(body_style 1)
 		(exclude_from_sim no)
-		(in_bom yes)
+		(in_bom no)
 		(on_board yes)
 		(in_pos_files yes)
@@
 		(body_style 1)
 		(exclude_from_sim no)
-		(in_bom yes)
+		(in_bom no)
 		(on_board yes)
 		(in_pos_files yes)
@@
 	)
 	(symbol
-		(lib_id "Connector:USB_C_Receptacle_PowerOnly_6P")
-		(at 35.56 43.18 0)
-		(unit 1)
-		(body_style 1)
-		(exclude_from_sim no)
-		(in_bom yes)
-		(on_board yes)
-		(in_pos_files yes)
-		(dnp no)
-		(fields_autoplaced yes)
-		(property "Reference" "J3"
-			(at 35.56 25.4 0)
-			(show_name no)
-			(do_not_autoplace no)
-			(effects
-				(font
-					(size 1.27 1.27)
-				)
-			)
-		)
-		(property "Value" "USB_C_Receptacle_PowerOnly_6P"
-			(at 35.56 27.94 0)
-			(show_name no)
-			(do_not_autoplace no)
-			(effects
-				(font
-					(size 1.27 1.27)
-				)
-			)
-		)
-		(property "Footprint" "Connector_USB:USB_C_Receptacle_GCT_USB4125-xx-x-0190_6P_TopMnt_Horizontal"
-			(at 39.37 40.64 0)
-			(hide yes)
-			(show_name no)
-			(do_not_autoplace no)
-			(effects
-				(font
-					(size 1.27 1.27)
-				)
-			)
-		)
-		(property "Datasheet" "https://www.usb.org/sites/default/files/documents/usb_type-c.zip"
-			(at 35.56 43.18 0)
-			(hide yes)
-			(show_name no)
-			(do_not_autoplace no)
-			(effects
-				(font
-					(size 1.27 1.27)
-				)
-			)
-		)
-		(property "Description" "USB Power-Only 6P Type-C Receptacle connector"
-			(at 35.56 43.18 0)
-			(hide yes)
-			(show_name no)
-			(do_not_autoplace no)
-			(effects
-				(font
-					(size 1.27 1.27)
-				)
-			)
-		)
-		(property "ID" "30"
-			(at 35.56 43.18 0)
-			(hide yes)
-			(show_name no)
-			(do_not_autoplace no)
-			(effects
-				(font
-					(size 1.27 1.27)
-				)
-			)
-		)
-		(property "Sim.Pins" ""
-			(at 35.56 43.18 0)
-			(hide yes)
-			(show_name no)
-			(do_not_autoplace no)
-			(effects
-				(font
-					(size 1.27 1.27)
-				)
-			)
-		)
-		(pin "A12"
-		)
-		(pin "S1"
-		)
-		(pin "B9"
-		)
-		(pin "A9"
-		)
-		(pin "B5"
-		)
-		(pin "B12"
-		)
-		(pin "A5"
-		)
-		(instances
-			(project "riaa_preamp"
-				(path "/2b990f77-15c8-4cc2-b07f-63b4e432ca20"
-					(reference "J3")
-					(unit 1)
-				)
-			)
-		)
-	)
-	(symbol
 		(lib_id "Device:R")
 		(at 127 170.18 90)
@@
 		(body_style 1)
 		(exclude_from_sim no)
-		(in_bom yes)
+		(in_bom no)
 		(on_board yes)
 		(in_pos_files yes)

Commit message: Finished with adding 9V Power Delivery
Parts:
- C17: ID (none) -> 93
- D3, D4: ID (none) -> 106
- J1, J2, J4, J5: ID (none) -> 52
- J3: ID (none) -> 30
- R18: ID (none) -> 97
- R2, R5: ID (none) -> 99
- R3, R6: ID (none) -> 98
- R46: ID (none) -> 96
- U1: ID (none) -> 100
- U2: ID (none) -> 101
- U3: ID (none) -> 102
- U4: ID (none) -> 103
Changed lines of the file:
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@@
 			)
 		)
+		(property "ID" "100"
+			(at 127 116.84 0)
+			(hide yes)
+			(show_name no)
+			(do_not_autoplace no)
+			(effects
+				(font
+					(size 1.27 1.27)
+				)
+			)
+		)
 		(pin "5"
 		)
@@
 			)
 		)
-		(property "ID" ""
+		(property "ID" "101"
 			(at 137.16 58.42 0)
 			(hide yes)
@@
 			)
 		)
+		(property "ID" "102"
+			(at 209.55 38.1 0)
+			(hide yes)
+			(show_name no)
+			(do_not_autoplace no)
+			(effects
+				(font
+					(size 1.27 1.27)
+				)
+			)
+		)
 		(pin "2"
 		)
@@
 			)
 		)
-		(property "ID" ""
+		(property "ID" "52"
 			(at 180.34 119.38 0)
 			(hide yes)
@@
 			)
 		)
+		(property "ID" "106"
+			(at 185.42 76.2 90)
+			(hide yes)
+			(show_name no)
+			(do_not_autoplace no)
+			(effects
+				(font
+					(size 1.27 1.27)
+				)
+			)
+		)
 		(pin "1"
 		)
@@
 			)
 		)
+		(property "ID" "100"
+			(at 127 160.02 0)
+			(hide yes)
+			(show_name no)
+			(do_not_autoplace no)
+			(effects
+				(font
+					(size 1.27 1.27)
+				)
+			)
+		)
 		(pin "1"
 		)
@@
 			)
 		)
+		(property "ID" "30"
+			(at 35.56 43.18 0)
+			(hide yes)
+			(show_name no)
+			(do_not_autoplace no)
+			(effects
+				(font
+					(size 1.27 1.27)
+				)
+			)
+		)
 		(pin "A5"
 		)
@@
 			)
 		)
+		(property "ID" "106"
+			(at 200.66 76.2 90)
+			(hide yes)
+			(show_name no)
+			(do_not_autoplace no)
+			(effects
+				(font
+					(size 1.27 1.27)
+				)
+			)
+		)
 		(pin "1"
 		)
@@
 			)
 		)
+		(property "ID" "98"
+			(at 100.33 82.55 0)
+			(hide yes)
+			(show_name no)
+			(do_not_autoplace no)
+			(effects
+				(font
+					(size 1.27 1.27)
+				)
+			)
+		)
 		(pin "2"
 		)
@@
 			)
 		)
+		(property "ID" "99"
+			(at 100.33 67.31 0)
+			(hide yes)
+			(show_name no)
+			(do_not_autoplace no)
+			(effects
+				(font
+					(size 1.27 1.27)
+				)
+			)
+		)
 		(pin "2"
 		)
@@
 			)
 		)
+		(property "ID" "103"
+			(at 266.7 40.64 0)
+			(hide yes)
+			(show_name no)
+			(do_not_autoplace no)
+			(effects
+				(font
+					(size 1.27 1.27)
+				)
+			)
+		)
 		(pin "1"
 		)
@@
 			)
 		)
+		(property "ID" "99"
+			(at 109.22 67.31 0)
+			(hide yes)
+			(show_name no)
+			(do_not_autoplace no)
+			(effects
+				(font
+					(size 1.27 1.27)
+				)
+			)
+		)
 		(pin "2"
 		)
@@
 			)
 		)
+		(property "ID" "93"
+			(at 231.14 38.1 0)
+			(hide yes)
+			(show_name no)
+			(do_not_autoplace no)
+			(effects
+				(font
+					(size 1.27 1.27)
+				)
+			)
+		)
 		(pin "1"
 		)
@@
 			)
 		)
+		(property "ID" "96"
+			(at 222.25 43.18 0)
+			(hide yes)
+			(show_name no)
+			(do_not_autoplace no)
+			(effects
+				(font
+					(size 1.27 1.27)
+				)
+			)
+		)
 		(pin "1"
 		)
@@
 			)
 		)
+		(property "ID" "100"
+			(at 212.09 130.81 0)
+			(hide yes)
+			(show_name no)
+			(do_not_autoplace no)
+			(effects
+				(font
+					(size 1.27 1.27)
+				)
+			)
+		)
 		(pin "8"
 		)
@@
 			)
 		)
-		(property "ID" ""
+		(property "ID" "52"
 			(at 22.86 116.84 0)
 			(hide yes)
@@
 			)
 		)
+		(property "ID" "98"
+			(at 109.22 82.55 0)
+			(hide yes)
+			(show_name no)
+			(do_not_autoplace no)
+			(effects
+				(font
+					(size 1.27 1.27)
+				)
+			)
+		)
 		(pin "2"
 		)
@@
 			)
 		)
+		(property "ID" "97"
+			(at 181.61 35.56 90)
+			(hide yes)
+			(show_name no)
+			(do_not_autoplace no)
+			(effects
+				(font
+					(size 1.27 1.27)
+				)
+			)
+		)
 		(pin "2"
 		)
@@
 			)
 		)
-		(property "ID" ""
+		(property "ID" "52"
 			(at 22.86 160.02 0)
 			(hide yes)
@@
 			)
 		)
-		(property "ID" ""
+		(property "ID" "52"
 			(at 180.34 162.56 0)
 			(hide yes)
